Commit message: Fix positions, colours, add fenders.

File: urdf/jackal.urdf.xacro (robot description, xacro)
@@ -2,8 +2,8 @@
 <robot name="robot" xmlns:xacro="http://www.ros.org/wiki/xacro">
   <!-- Constants for robot dimensions -->
-  <xacro:property name="PI" value="3.1415926535897931"/>
+  <xacro:property name="PI" value="3.1415926535897931" />
   <xacro:property name="wheelbase" value="0.240" />
   <xacro:property name="track" value="0.37559" />
-  <xacro:property name="wheel_vertical_offset" value="-0.0345" />
+  <xacro:property name="wheel_vertical_offset" value="0.0345" />
   <xacro:property name="base_stl_vertical_offset" value="-0.0655" />
   <xacro:property name="wheel_radius" value="0.098" />
@@ -12,4 +12,7 @@
   <xacro:property name="chassis_width" value="0.310" />
   <xacro:property name="chassis_height" value="0.184" />
+  <material name="dark_grey"><color rgba="0.2 0.2 0.2 1.0" /></material>
+  <material name="yellow"><color rgba="0.8 0.8 0.0 1.0" /></material>
+  <material name="black"><color rgba="0.15 0.15 0.15 1.0" /></material>
   <xacro:macro name="wheel" params="prefix *joint_pose">
     <link name="${prefix}_wheel">
@@ -20,8 +23,9 @@
       </inertial>
       <visual>
-        <origin xyz="0 0 0" rpy="0 0 0"/>
+        <origin xyz="0 0 0" rpy="${PI/2} 0 0"/>
         <geometry>
           <mesh filename="package://jackal_description/meshes/jackal-wheel.stl"/>
         </geometry>
+        <material name="black" />
       </visual>
       <collision>
@@ -34,7 +38,7 @@
     <joint name="${prefix}_wheel_joint" type="continuous">
       <parent link="base_link"/>
-      <child link="${prefix}_wheel"/>
-      <xacro:insert_block name="joint_pose"/>
-      <axis xyz="0 1 0"/>
+      <child link="${prefix}_wheel" />
+      <xacro:insert_block name="joint_pose" />
+      <axis xyz="0 1 0" />
     </joint>
     <gazebo reference="${prefix}_wheel">
@@ -44,29 +48,30 @@
   </xacro:macro>
   <xacro:wheel prefix="front_left">
-    <origin xyz="${track/2} ${wheelbase/2} ${wheel_vertical_offset}" rpy="0 0 0"/>
+    <origin xyz="${wheelbase/2} ${track/2} ${wheel_vertical_offset}" rpy="0 0 0" />
   </xacro:wheel>
   <xacro:wheel prefix="front_right">
-    <origin xyz="${track/2} ${-wheelbase/2} ${wheel_vertical_offset}" rpy="0 0 0"/>
+    <origin xyz="${wheelbase/2} ${-track/2} ${wheel_vertical_offset}" rpy="0 0 0" />
   </xacro:wheel>
   <xacro:wheel prefix="rear_left">
-    <origin xyz="${-track/2} ${wheelbase/2} ${wheel_vertical_offset}" rpy="0 0 0"/>
+    <origin xyz="${-wheelbase/2} ${track/2} ${wheel_vertical_offset}" rpy="0 0 0" />
   </xacro:wheel>
   <xacro:wheel prefix="rear_right">
-    <origin xyz="${-track/2} ${-wheelbase/2} ${wheel_vertical_offset}" rpy="0 0 0"/>
+    <origin xyz="${-wheelbase/2} ${-track/2} ${wheel_vertical_offset}" rpy="0 0 0" />
   </xacro:wheel>
   <link name="base_link">
     <inertial>
-      <origin xyz="0 0 0" rpy="0 0 0"/>
-      <mass value="20"/>
-      <inertia ixx="1" ixy="0" ixz="0" iyy="1" iyz="0" izz="1"/>
+      <origin xyz="0 0 0" rpy="0 0 0" />
+      <mass value="20" />
+      <inertia ixx="1" ixy="0" ixz="0" iyy="1" iyz="0" izz="1" />
     </inertial>
     <visual>
-      <origin xyz="0 0 0" rpy="0 0 0"/>
+      <origin xyz="0 0 ${base_stl_vertical_offset}" rpy="${PI/2} 0 ${PI/2}"/>
       <geometry>
         <mesh filename="package://jackal_description/meshes/jackal-base.stl"/>
       </geometry>
+      <material name="dark_grey" />
     </visual>
     <collision>
-      <origin xyz="0 0 0"/>
+      <origin xyz="0 0 ${chassis_height/2}"/>
       <geometry>
         <box size="${chassis_length} ${chassis_width} ${chassis_height}"/>
@@ -77,26 +82,18 @@
     <selfCollide>false</selfCollide>
   </gazebo>
-  <!-- <link name="base_link">
-    <inertial>
-      <origin xyz="0 0 0" rpy="0 0 0"/>
-      <mass value="20"/>
-      <inertia ixx="1" ixy="0" ixz="0" iyy="1" iyz="0" izz="1"/>
-    </inertial>
+  <link name="fenders_link">
     <visual>
-      <origin xyz="0 0 0" rpy="0 0 0"/>
+      <origin xyz="0 0 ${base_stl_vertical_offset}" rpy="${PI/2} 0 ${PI/2}"/>
       <geometry>
-        <mesh filename="$(find jackal_description)/meshes/jackal-base.stl"/>
+        <mesh filename="package://jackal_description/meshes/jackal-fenders.stl"/>
       </geometry>
+      <material name="yellow" />
     </visual>
-    <collision>
-      <origin xyz="0 0 0"/>
-      <geometry>
-        <box size="${chassis_length} ${chassis_width} ${chassis_height}"/>
-      </geometry>
-    </collision>
   </link>
-  <gazebo reference="base_link">
-    <selfCollide>false</selfCollide>
-  </gazebo> -->
+  <joint name="$fenders_joint" type="fixed">
+    <parent link="base_link" />
+    <child link="fenders_link" />
+    <origin xyz="0 0 0" />
+  </joint>
   <!-- <gazebo>
     <plugin name="" filename="">

Commit message: Remove invalid inertial info, add mount points.

File: urdf/jackal.urdf.xacro (robot description, xacro)
@@ -1,10 +1,9 @@
 <?xml version="1.0"?>
 <robot name="robot" xmlns:xacro="http://www.ros.org/wiki/xacro">
-  <!-- Constants for robot dimensions -->
   <xacro:property name="PI" value="3.1415926535897931" />
   <xacro:property name="wheelbase" value="0.240" />
   <xacro:property name="track" value="0.37559" />
   <xacro:property name="wheel_vertical_offset" value="0.0345" />
-  <xacro:property name="base_stl_vertical_offset" value="-0.0655" />
+  <xacro:property name="footprint_vertical_offset" value="-0.0655" />
   <xacro:property name="wheel_radius" value="0.098" />
   <xacro:property name="wheel_width" value="0.040" />
@@ -12,4 +11,6 @@
   <xacro:property name="chassis_width" value="0.310" />
   <xacro:property name="chassis_height" value="0.184" />
+  <xacro:property name="mount_spacing" value="0.120" />
+  <xacro:property name="mount_standoff_height" value="0.0075" />
   <material name="dark_grey"><color rgba="0.2 0.2 0.2 1.0" /></material>
   <material name="yellow"><color rgba="0.8 0.8 0.0 1.0" /></material>
@@ -17,9 +18,4 @@
   <xacro:macro name="wheel" params="prefix *joint_pose">
     <link name="${prefix}_wheel">
-      <inertial>
-        <origin xyz="0 0 0" rpy="0 0 0"/>
-        <mass value="100"/>
-        <inertia ixx="0.2" ixy="0" ixz="0" iyy="0.2" iyz="0" izz="0.2"/>
-      </inertial>
       <visual>
         <origin xyz="0 0 0" rpy="${PI/2} 0 0"/>
@@ -42,8 +38,4 @@
       <axis xyz="0 1 0" />
     </joint>
-    <gazebo reference="${prefix}_wheel">
-      <material>Gazebo/Yellow</material>
-      <selfCollide>false</selfCollide>
-    </gazebo>
   </xacro:macro>
   <xacro:wheel prefix="front_left">
@@ -60,11 +52,6 @@
   </xacro:wheel>
   <link name="base_link">
-    <inertial>
-      <origin xyz="0 0 0" rpy="0 0 0" />
-      <mass value="20" />
-      <inertia ixx="1" ixy="0" ixz="0" iyy="1" iyz="0" izz="1" />
-    </inertial>
     <visual>
-      <origin xyz="0 0 ${base_stl_vertical_offset}" rpy="${PI/2} 0 ${PI/2}"/>
+      <origin xyz="0 0 ${footprint_vertical_offset}" rpy="${PI/2} 0 ${PI/2}"/>
       <geometry>
         <mesh filename="package://jackal_description/meshes/jackal-base.stl"/>
@@ -79,10 +66,7 @@
     </collision>
   </link>
-  <gazebo reference="base_link">
-    <selfCollide>false</selfCollide>
-  </gazebo>
   <link name="fenders_link">
     <visual>
-      <origin xyz="0 0 ${base_stl_vertical_offset}" rpy="${PI/2} 0 ${PI/2}"/>
+      <origin xyz="0 0 ${footprint_vertical_offset}" rpy="${PI/2} 0 ${PI/2}"/>
       <geometry>
         <mesh filename="package://jackal_description/meshes/jackal-fenders.stl"/>
@@ -96,14 +80,21 @@
     <origin xyz="0 0 0" />
   </joint>
-  <!-- <gazebo>
-    <plugin name="" filename="">
-      <alwaysOn>true</alwaysOn>
-      <updateRate>100.0</updateRate>
-      <leftJoint>left_wheel_jnt</leftJoint>
-      <rightJoint>right_wheel_jnt</rightJoint>
-      <wheelSeparation>${axle}</wheelSeparation>
-      <wheelDiameter>${wheel_radius*2}</wheelDiameter>
-      <torque>35</torque>
-    </plugin>
-  </gazebo> -->
+  <link name="mid_mount"></link>
+  <joint name="mid_mount_joint" type="fixed">
+    <parent link="base_link" />
+    <child link="mid_mount" />
+    <origin xyz="0 0 ${chassis_height+mount_standoff_height}" />
+  </joint>
+  <link name="rear_mount"></link>
+  <joint name="rear_mount_joint" type="fixed">
+    <parent link="mid_mount" />
+    <child link="rear_mount" />
+    <origin xyz="${-mount_spacing} 0 0" />
+  </joint>
+  <link name="front_mount"></link>
+  <joint name="front_mount_joint" type="fixed">
+    <parent link="mid_mount" />
+    <child link="front_mount" />
+    <origin xyz="${mount_spacing} 0 0" />
+  </joint>
 </robot>

Commit message: Add navsat_link and imu_link.

File: urdf/jackal.urdf.xacro (robot description, xacro)
@@ -80,4 +80,29 @@
     <origin xyz="0 0 0" />
   </joint>
+  <!-- TODO: Make this internal_imu_link or something, and use a mixed-in xacro
+       to supply the joint between it and imu_link. This is important so that imu_link
+       always points to the "active" IMU. When an upgrade IMU is connected, the
+       internal_imu_link should remain, but imu_link should point to the upgrade one. -->
+  <link name="imu_link"></link>
+  <joint name="imu_joint" type="fixed">
+    <parent link="base_link" />
+    <child link="imu_link" />
+    <origin xyz="-0.1974 0.0314 0.163" />
+  </joint>
+  <!-- TODO: Same note as applies to imu_link -->
+  <link name="navsat_link">
+    <visual>
+      <geometry>
+        <cylinder radius="0.026" length="0.016" />
+      </geometry>
+      <origin xyz="0 0 0.008" />
+      <material name="black" />
+    </visual>
+  </link>
+  <joint name="navsat_joint" type="fixed">
+    <parent link="base_link" />
+    <child link="navsat_link" />
+    <origin xyz="-0.180 0.126 0.1815" />
+  </joint>
   <link name="mid_mount"></link>
   <joint name="mid_mount_joint" type="fixed">

Commit message: Update description with v0.9 hardware changes.

File: urdf/jackal.urdf.xacro (robot description, xacro)
@@ -2,5 +2,5 @@
 <robot name="robot" xmlns:xacro="http://www.ros.org/wiki/xacro">
   <xacro:property name="PI" value="3.1415926535897931" />
-  <xacro:property name="wheelbase" value="0.240" />
+  <xacro:property name="wheelbase" value="0.262" />
   <xacro:property name="track" value="0.37559" />
   <xacro:property name="wheel_vertical_offset" value="0.0345" />
@@ -12,5 +12,4 @@
   <xacro:property name="chassis_height" value="0.184" />
   <xacro:property name="mount_spacing" value="0.120" />
-  <xacro:property name="mount_standoff_height" value="0.0075" />
   <material name="dark_grey"><color rgba="0.2 0.2 0.2 1.0" /></material>
   <material name="yellow"><color rgba="0.8 0.8 0.0 1.0" /></material>
@@ -109,5 +108,5 @@
     <parent link="base_link" />
     <child link="mid_mount" />
-    <origin xyz="0 0 ${chassis_height+mount_standoff_height}" />
+    <origin xyz="0 0 ${chassis_height}" />
   </joint>
   <link name="rear_mount"></link>

Commit message: Add provisional sim data to description.

File: urdf/jackal.urdf.xacro (robot description, xacro)
@@ -1,4 +1,4 @@
 <?xml version="1.0"?>
-<robot name="robot" xmlns:xacro="http://www.ros.org/wiki/xacro">
+<robot name="jackal" xmlns:xacro="http://www.ros.org/wiki/xacro">
   <xacro:property name="PI" value="3.1415926535897931" />
   <xacro:property name="wheelbase" value="0.262" />
@@ -16,5 +16,5 @@
   <material name="black"><color rgba="0.15 0.15 0.15 1.0" /></material>
   <xacro:macro name="wheel" params="prefix *joint_pose">
-    <link name="${prefix}_wheel">
+    <link name="${prefix}_wheel_link">
       <visual>
         <origin xyz="0 0 0" rpy="${PI/2} 0 0"/>
@@ -30,11 +30,33 @@
         </geometry>
       </collision>
+      <inertial>
+        <origin xyz="0 0 0" rpy="0 0 0"/>
+        <mass value="0.6"/>
+        <inertia
+          ixx="1.0" ixy="0.0" ixz="0.0"
+          iyy="1.0" iyz="0.0"
+          izz="1.0"/>
+      </inertial>
     </link>
-    <joint name="${prefix}_wheel_joint" type="continuous">
+    <gazebo reference="${prefix}_wheel_link">
+      <material>Gazebo/DarkGrey</material>
+    </gazebo>
+    <joint name="${prefix}_wheel" type="continuous">
       <parent link="base_link"/>
-      <child link="${prefix}_wheel" />
+      <child link="${prefix}_wheel_link" />
       <xacro:insert_block name="joint_pose" />
       <axis xyz="0 1 0" />
     </joint>
+    <!-- In reality, Jackal has only two motors, one per side. However, it's more
+         straightforward for Gazebo to simulate as if there's on actuator per wheel. -->
+    <transmission name="${prefix}_wheel_trans">
+      <type>transmission_interface/SimpleTransmission</type>
+      <joint name="${prefix}_wheel">
+        <hardwareInterface>VelocityJointInterface</hardwareInterface>
+      </joint>
+      <actuator name="${prefix}_actuator">
+        <mechanicalReduction>1</mechanicalReduction>
+      </actuator>
+    </transmission>
   </xacro:macro>
   <xacro:wheel prefix="front_left">
@@ -64,4 +86,12 @@
       </geometry>
     </collision>
+    <inertial>
+      <origin xyz="0 0 ${chassis_height/2}" rpy="0 0 0"/>
+      <mass value="16"/>
+      <inertia
+        ixx="1.0" ixy="0.0" ixz="0.0"
+        iyy="1.0" iyz="0.0"
+        izz="1.0"/>
+      </inertial>
   </link>
   <link name="fenders_link">
@@ -74,5 +104,5 @@
     </visual>
   </link>
-  <joint name="$fenders_joint" type="fixed">
+  <joint name="fenders_joint" type="fixed">
     <parent link="base_link" />
     <child link="fenders_link" />
@@ -122,3 +152,5 @@
     <origin xyz="${mount_spacing} 0 0" />
   </joint>
+  <!-- Bring in simulation data for Gazebo -->
+  <xacro:include filename="jackal.gazebo" />
 </robot>

Commit message: fixed inertia parameters. added imu plugin--not working

File: urdf/jackal.urdf.xacro (robot description, xacro)
@@ -8,7 +8,22 @@
   <xacro:property name="wheel_radius" value="0.098" />
   <xacro:property name="wheel_width" value="0.040" />
+  <xacro:property name="wheel_mass" value="0.477"/>
+  <xacro:property name="wheel_ixx" value="1253420.30e-09"/>
+  <xacro:property name="wheel_ixy" value="0.00"/>
+  <xacro:property name="wheel_ixz" value="0.00"/>
+  <xacro:property name="wheel_iyy" value="1253462.44e-09"/>
+  <xacro:property name="wheel_iyz" value="18.77e-09"/>
+  <xacro:property name="wheel_izz" value="2358919.20e-09"/>
   <xacro:property name="chassis_length" value="0.420" />
   <xacro:property name="chassis_width" value="0.310" />
   <xacro:property name="chassis_height" value="0.184" />
+  <xacro:property name="chassis_mass" value="16523.98e-03"/>
+  <xacro:property name="chassis_ixx" value="392236674.19e-09"/>
+  <xacro:property name="chassis_ixy" value="-856992.99e-09"/>
+  <xacro:property name="chassis_ixz" value="-782275.61e-09"/>
+  <xacro:property name="chassis_iyy" value="448518333.08e-09"/>
+  <xacro:property name="chassis_iyz" value="16413049.38e-09"/>
+  <xacro:property name="chassis_izz" value="313604474.79e-09"/>
+  <xacro:property name="dummy_inertia" value="1e-09"/>
   <xacro:property name="mount_spacing" value="0.120" />
   <material name="dark_grey"><color rgba="0.2 0.2 0.2 1.0" /></material>
@@ -31,10 +46,10 @@
       </collision>
       <inertial>
-        <origin xyz="0 0 0" rpy="0 0 0"/>
-        <mass value="0.6"/>
+        <origin xyz="0.0 0.0 0.0" rpy="0 0 0"/>
+        <mass value="${wheel_mass}"/>
         <inertia
-          ixx="1.0" ixy="0.0" ixz="0.0"
-          iyy="1.0" iyz="0.0"
-          izz="1.0"/>
+          ixx="${wheel_ixx}" ixy="${wheel_ixy}" ixz="${wheel_ixz}"
+          iyy="${wheel_iyy}" iyz="${wheel_iyz}"
+          izz="${wheel_izz}"/>
       </inertial>
     </link>
@@ -75,4 +90,5 @@
     <visual>
       <origin xyz="0 0 ${footprint_vertical_offset}" rpy="${PI/2} 0 ${PI/2}"/>
+      <!-- <origin xyz="0 0 ${chassis_height/2}" rpy="${PI/2} 0 ${PI/2}"/> -->
       <geometry>
         <mesh filename="package://jackal_description/meshes/jackal-base.stl"/>
@@ -88,9 +104,10 @@
     <inertial>
       <origin xyz="0 0 ${chassis_height/2}" rpy="0 0 0"/>
-      <mass value="16"/>
+      <!-- <origin xyz="1.91e-03 66.60e-03 11.92e-03" rpy="0 0 0"/> -->
+      <mass value="${chassis_mass}"/>
       <inertia
-        ixx="1.0" ixy="0.0" ixz="0.0"
-        iyy="1.0" iyz="0.0"
-        izz="1.0"/>
+        ixx="${chassis_ixx}" ixy="${chassis_ixy}" ixz="${chassis_ixz}"
+        iyy="${chassis_iyy}" iyz="${chassis_iyz}"
+        izz="${chassis_izz}"/>
       </inertial>
   </link>
@@ -98,4 +115,5 @@
     <visual>
       <origin xyz="0 0 ${footprint_vertical_offset}" rpy="${PI/2} 0 ${PI/2}"/>
+      <!-- <origin xyz="0 0 ${chassis_height/2}" rpy="${PI/2} 0 ${PI/2}"/> -->
       <geometry>
         <mesh filename="package://jackal_description/meshes/jackal-fenders.stl"/>
@@ -113,5 +131,12 @@
        always points to the "active" IMU. When an upgrade IMU is connected, the
        internal_imu_link should remain, but imu_link should point to the upgrade one. -->
-  <link name="imu_link"></link>
+  <link name="imu_link">
+    <inertial>
+      <mass value="0.001"/>
+      <!-- <origin xyz="-0.1974 0.0314 0.163" rpy="0 0 0"/> -->
+      <origin xyz="0 0 0" rpy="0 0 0"/>
+      <inertia ixx="${dummy_inertia}" ixy="0.0" ixz="0.0" iyy="${dummy_inertia}" iyz="0.0" izz="${dummy_inertia}"/>
+    </inertial>
+  </link>
   <joint name="imu_joint" type="fixed">
     <parent link="base_link" />

Commit message: changed some physical and collision properties.

File: urdf/jackal.urdf.xacro (robot description, xacro)
@@ -8,21 +8,7 @@
   <xacro:property name="wheel_radius" value="0.098" />
   <xacro:property name="wheel_width" value="0.040" />
-  <xacro:property name="wheel_mass" value="0.477"/>
-  <xacro:property name="wheel_ixx" value="1253420.30e-09"/>
-  <xacro:property name="wheel_ixy" value="0.00"/>
-  <xacro:property name="wheel_ixz" value="0.00"/>
-  <xacro:property name="wheel_iyy" value="1253462.44e-09"/>
-  <xacro:property name="wheel_iyz" value="18.77e-09"/>
-  <xacro:property name="wheel_izz" value="2358919.20e-09"/>
   <xacro:property name="chassis_length" value="0.420" />
   <xacro:property name="chassis_width" value="0.310" />
   <xacro:property name="chassis_height" value="0.184" />
-  <xacro:property name="chassis_mass" value="16523.98e-03"/>
-  <xacro:property name="chassis_ixx" value="392236674.19e-09"/>
-  <xacro:property name="chassis_ixy" value="-856992.99e-09"/>
-  <xacro:property name="chassis_ixz" value="-782275.61e-09"/>
-  <xacro:property name="chassis_iyy" value="448518333.08e-09"/>
-  <xacro:property name="chassis_iyz" value="16413049.38e-09"/>
-  <xacro:property name="chassis_izz" value="313604474.79e-09"/>
   <xacro:property name="dummy_inertia" value="1e-09"/>
   <xacro:property name="mount_spacing" value="0.120" />
@@ -46,10 +32,10 @@
       </collision>
       <inertial>
-        <origin xyz="0.0 0.0 0.0" rpy="0 0 0"/>
-        <mass value="${wheel_mass}"/>
+        <origin xyz="-0.0001 0 -0.00001" rpy="0 0 0"/>
+        <mass value="0.477"/>
         <inertia
-          ixx="${wheel_ixx}" ixy="${wheel_ixy}" ixz="${wheel_ixz}"
-          iyy="${wheel_iyy}" iyz="${wheel_iyz}"
-          izz="${wheel_izz}"/>
+          ixx="0.0024" ixy="0" ixz="0"
+          iyy="0.0013" iyz="0"
+          izz="0.0013"/>
       </inertial>
     </link>
@@ -58,5 +44,5 @@
     </gazebo>
     <joint name="${prefix}_wheel" type="continuous">
-      <parent link="base_link"/>
+      <parent link="chassis_link"/>
       <child link="${prefix}_wheel_link" />
       <xacro:insert_block name="joint_pose" />
@@ -64,5 +50,5 @@
     </joint>
     <!-- In reality, Jackal has only two motors, one per side. However, it's more
-         straightforward for Gazebo to simulate as if there's on actuator per wheel. -->
+         straightforward for Gazebo to simulate as if there's an actuator per wheel. -->
     <transmission name="${prefix}_wheel_trans">
       <type>transmission_interface/SimpleTransmission</type>
@@ -88,7 +74,26 @@
   </xacro:wheel>
   <link name="base_link">
+    <inertial>
+      <mass value="0.0001" />
+      <origin xyz="0 0 0" />
+      <inertia  ixx="0.0001" ixy="0.0" ixz="0.0"
+                iyy="0.0001" iyz="0.0"
+                izz="0.0001" />
+    </inertial>
+    <visual>
+      <origin xyz="0 0 0" rpy="0 0 0" />
+      <geometry>
+      <box size="0.001 0.001 0.001" />
+    </geometry>
+    </visual>
+  </link>
+  <joint name="base_link_joint" type="fixed">
+    <origin xyz="0 0 0" rpy="0 0 0" />
+    <parent link="base_link"/>
+    <child link="chassis_link" />
+  </joint>
+  <link name="chassis_link">
     <visual>
       <origin xyz="0 0 ${footprint_vertical_offset}" rpy="${PI/2} 0 ${PI/2}"/>
-      <!-- <origin xyz="0 0 ${chassis_height/2}" rpy="${PI/2} 0 ${PI/2}"/> -->
       <geometry>
         <mesh filename="package://jackal_description/meshes/jackal-base.stl"/>
@@ -103,11 +108,12 @@
     </collision>
     <inertial>
-      <origin xyz="0 0 ${chassis_height/2}" rpy="0 0 0"/>
-      <!-- <origin xyz="1.91e-03 66.60e-03 11.92e-03" rpy="0 0 0"/> -->
-      <mass value="${chassis_mass}"/>
+      <!-- Center of mass -->
+      <origin xyz="0.012  0.002 0.067" rpy="0 0 0"/>
+      <mass value="16.523"/>
+      <!-- Moments of inertia: ( chassis without wheels ) -->
       <inertia
-        ixx="${chassis_ixx}" ixy="${chassis_ixy}" ixz="${chassis_ixz}"
-        iyy="${chassis_iyy}" iyz="${chassis_iyz}"
-        izz="${chassis_izz}"/>
+        ixx="0.3136" ixy="-0.0008" ixz="0.0164"
+        iyy="0.3922" iyz="-0.0009"
+        izz="0.4485"/>
       </inertial>
   </link>
@@ -115,5 +121,4 @@
     <visual>
       <origin xyz="0 0 ${footprint_vertical_offset}" rpy="${PI/2} 0 ${PI/2}"/>
-      <!-- <origin xyz="0 0 ${chassis_height/2}" rpy="${PI/2} 0 ${PI/2}"/> -->
       <geometry>
         <mesh filename="package://jackal_description/meshes/jackal-fenders.stl"/>
@@ -123,7 +128,6 @@
   </link>
   <joint name="fenders_joint" type="fixed">
-    <parent link="base_link" />
+    <parent link="chassis_link" />
     <child link="fenders_link" />
-    <origin xyz="0 0 0" />
   </joint>
   <!-- TODO: Make this internal_imu_link or something, and use a mixed-in xacro
@@ -134,5 +138,4 @@
     <inertial>
       <mass value="0.001"/>
-      <!-- <origin xyz="-0.1974 0.0314 0.163" rpy="0 0 0"/> -->
       <origin xyz="0 0 0" rpy="0 0 0"/>
       <inertia ixx="${dummy_inertia}" ixy="0.0" ixz="0.0" iyy="${dummy_inertia}" iyz="0.0" izz="${dummy_inertia}"/>
@@ -140,7 +143,6 @@
   </link>
   <joint name="imu_joint" type="fixed">
-    <parent link="base_link" />
+    <parent link="chassis_link" />
     <child link="imu_link" />
-    <origin xyz="-0.1974 0.0314 0.163" />
   </joint>
   <!-- TODO: Same note as applies to imu_link -->
@@ -155,5 +157,5 @@
   </link>
   <joint name="navsat_joint" type="fixed">
-    <parent link="base_link" />
+    <parent link="chassis_link" />
     <child link="navsat_link" />
     <origin xyz="-0.180 0.126 0.1815" />
@@ -161,5 +163,5 @@
   <link name="mid_mount"></link>
   <joint name="mid_mount_joint" type="fixed">
-    <parent link="base_link" />
+    <parent link="chassis_link" />
     <child link="mid_mount" />
     <origin xyz="0 0 ${chassis_height}" />
