Commit message: Add front laser accessory to description.

File: urdf/jackal.urdf.xacro (robot description, xacro)
@@ -14,4 +14,5 @@
   <xacro:property name="mount_spacing" value="0.120" />
   <material name="dark_grey"><color rgba="0.2 0.2 0.2 1.0" /></material>
+  <material name="light_grey"><color rgba="0.4 0.4 0.4 1.0" /></material>
   <material name="yellow"><color rgba="0.8 0.8 0.0 1.0" /></material>
   <material name="black"><color rgba="0.15 0.15 0.15 1.0" /></material>
@@ -181,3 +182,6 @@
   <!-- Bring in simulation data for Gazebo -->
   <xacro:include filename="jackal.gazebo" />
+  <xacro:if value="$(arg accessories)">
+    <xacro:include filename="accessories.urdf.xacro" />
+  </xacro:if>
 </robot>

Commit message: Removed inertial and geometry of the base_link.

File: urdf/jackal.urdf.xacro (robot description, xacro)
@@ -74,19 +74,5 @@
     <origin xyz="${-wheelbase/2} ${-track/2} ${wheel_vertical_offset}" rpy="0 0 0" />
   </xacro:wheel>
-  <link name="base_link">
-    <inertial>
-      <mass value="0.0001" />
-      <origin xyz="0 0 0" />
-      <inertia  ixx="0.0001" ixy="0.0" ixz="0.0"
-                iyy="0.0001" iyz="0.0"
-                izz="0.0001" />
-    </inertial>
-    <visual>
-      <origin xyz="0 0 0" rpy="0 0 0" />
-      <geometry>
-      <box size="0.001 0.001 0.001" />
-    </geometry>
-    </visual>
-  </link>
+  <link name="base_link"></link>
   <joint name="base_link_joint" type="fixed">
     <origin xyz="0 0 0" rpy="0 0 0" />

Commit message: Fix wheel inertia, based on Gazebo 5 inertia visualization.

File: urdf/jackal.urdf.xacro (robot description, xacro)
@@ -33,9 +33,9 @@
       </collision>
       <inertial>
-        <origin xyz="-0.0001 0 -0.00001" rpy="0 0 0"/>
+        <origin xyz="0 0 0" rpy="0 0 0"/>
         <mass value="0.477"/>
         <inertia
-          ixx="0.0024" ixy="0" ixz="0"
-          iyy="0.0013" iyz="0"
+          ixx="0.0013" ixy="0" ixz="0"
+          iyy="0.0024" iyz="0"
           izz="0.0013"/>
       </inertial>

Commit message: Removed unused variable jackal_description_dir

File: urdf/jackal.urdf.xacro (robot description, xacro)
@@ -13,5 +13,4 @@
   <xacro:property name="dummy_inertia" value="1e-09"/>
   <xacro:property name="mount_spacing" value="0.120" />
-  <xacro:property name="jackal_description_dir" value="$(find jackal_description)" />
   <material name="dark_grey"><color rgba="0.2 0.2 0.2 1.0" /></material>
   <material name="light_grey"><color rgba="0.4 0.4 0.4 1.0" /></material>

Commit message: Added Microstrain GX5 to description

File: urdf/jackal.urdf.xacro (robot description, xacro)
@@ -203,4 +203,16 @@
     <origin xyz="-0.180 0.126 0.1815" />
   </joint>
+  <!--
+    Optionally add a GX5 IMU
+  -->
+  <xacro:if value="$(optenv JACKAL_GX5_IMU 0)">
+    <link name="gx5_link" />
+    <joint name="gx5_joint" type="fixed">
+      <parent link="$(optenv JACKAL_GX5_IMU_PARENT base_link)" />
+      <child link="gx5_link" />
+      <!-- TODO This offset & rotation may not be final, but it's good enough for now.  May update, pending RSCI-10 -->
+      <origin xyz="$(optenv JACKAL_GX5_IMU_OFFSET -0.139 0.096 0.100)" rpy="$(optenv JACKAL_GX5_IMU_RPY ${PI} 0 -${PI/2})" />
+    </joint>
+  </xacro:if>
   <link name="mid_mount"></link>
   <joint name="mid_mount_joint" type="fixed">
@@ -229,3 +241,5 @@
   <!-- Optional custom includes. -->
   <xacro:include filename="$(optenv JACKAL_URDF_EXTRAS empty.urdf)" />
+  <!-- Optional for Clearpath internal softwares -->
+  <xacro:include filename="$(optenv CPR_URDF_EXTRAS empty.urdf)" />
 </robot>
