Commit message: Switch to parameterizing URDF with optenv.

File: urdf/accessories.urdf.xacro (robot description, xacro)
@@ -2,21 +2,23 @@
 <robot xmlns:xacro="http://www.ros.org/wiki/xacro">
   <!--
-    As you add args to this xacro, please ensure that they
-    are included with default values in each of the following
-    launch files:
+    As you add to this xacro, please be aware that both the robot and
+    simulation include it. You must retain compatibility with all of
+    the following launch files:
     jackal_viz/launch/view_model.launch
     jackal_gazebo/launch/jackal_world.launch
     jackal_base/launch/base.launch
   -->
-  <xacro:include filename="accessories/sick_lms100.urdf.xacro" />
-  <xacro:include filename="accessories/point_grey_flea.urdf.xacro" />
-  <xacro:if value="$(arg front_laser)">
-    <xacro:sick_lms100 prefix="front" />
-    <joint name="front_laser_joint" type="fixed">
-      <origin xyz="0.04 0 0.04" rpy="${PI} 0 0" />
-      <parent link="front_mount" />
-      <child link="front_laser" />
+  <xacro:include filename="accessories/sick_lms1xx.urdf.xacro" />
+  <xacro:if value="$(optenv JACKAL_LASER 0)">
+    <sick_lms1xx_mount prefix="$(optenv JACKAL_LASER_MOUNT front)" />
+    <joint name="$front_laser_mount_joint" type="fixed">
+      <origin xyz="$(optenv JACKAL_LASER_OFFSET 0 0 0)"
+              rpy="$(optenv JACKAL_LASER_RPY 0 0 0)" />
+      <parent link="$(optenv JACKAL_LASER_MOUNT front)_mount" />
+      <child link="$(optenv JACKAL_LASER_MOUNT front)_laser_mount" />
     </joint>
   </xacro:if>
+  <!--
+  <xacro:include filename="accessories/point_grey_flea.urdf.xacro" />
   <xacro:if value="$(arg camera)">
     <xacro:point_grey_flea3
@@ -39,3 +41,4 @@
       />
   </xacro:if>
+  -->
 </robot>

File: urdf/accessories/sick_lms1xx.urdf.xacro (robot description, xacro)
@@ -2,5 +2,5 @@
 <!--
 Copyright (c) 2013, Goncalo Cabrita, ISR University of Coimbra
-Copyright (c) 2014, Clearpath Robotics
+Copyright (c) 2014, 2015 Clearpath Robotics
 All rights reserved.
 Redistribution and use in source and binary forms, with or without
@@ -25,5 +25,5 @@
 SOFTWARE, EVEN IF ADVISED OF THE POSSIBILITY OF SUCH DAMAGE.
 -->
-<robot  xmlns:xacro="http://ros.org/wiki/xacro" name="sick_lms100">
+<robot xmlns:xacro="http://ros.org/wiki/xacro">
   <xacro:property name="laser_x" value="0.105" />
   <xacro:property name="laser_y" value="0.102" />
@@ -39,5 +39,15 @@
     </inertial>
   </xacro:macro>
-  <xacro:macro name="sick_lms100" params="prefix">
+  <xacro:macro name="sick_lms1xx_mount" params="prefix">
+    <link name="${prefix}_laser_mount">
+      <visual>
+        <origin xyz="0 0 0" rpy="0 0 0" />
+        <geometry>
+          <!-- Origin of this mesh is the base of the bracket. -->
+          <mesh filename="package://jackal_description/meshes/sick-lms1xx-bracket.stl" />
+        </geometry>
+        <material name="dark_grey" />
+      </visual>
+    </link>
     <link name="${prefix}_laser">
       <xacro:box_inertial x="${laser_x}" y="${laser_y}" z="${laser_z}" mass="${laser_mass}" />
@@ -45,5 +55,6 @@
         <origin xyz="0 0 0" rpy="0 0 0" />
         <geometry>
-          <mesh filename="package://jackal_description/meshes/sick_lms100.stl" />
+          <!-- Origin of this mesh is the focal point of the LIDAR. -->
+          <mesh filename="package://jackal_description/meshes/sick-lms1xx.stl" />
         </geometry>
         <material name="light_grey" />
@@ -56,4 +67,10 @@
       </collision>
     </link>
+    <joint name="${prefix}_laser_joint" type="fixed">
+      <!-- This offset is from the base of the bracket to the LIDAR's focal point. -->
+      <origin xyz="0 0 0.149" rpy="0 0 0" />
+      <parent link="${prefix}_laser_mount" />
+      <child link="${prefix}_laser" />
+    </joint>
     <gazebo reference="${prefix}_laser">
       <material>Gazebo/Grey</material>

File: urdf/jackal.urdf.xacro (robot description, xacro)
@@ -166,8 +166,9 @@
     <origin xyz="${mount_spacing} 0 0" />
   </joint>
-  <!-- Bring in simulation data for Gazebo -->
+  <!-- Bring in simulation data for Gazebo. -->
   <xacro:include filename="jackal.gazebo" />
-  <xacro:if value="$(arg accessories)">
-    <xacro:include filename="accessories.urdf.xacro" />
-  </xacro:if>
+  <!-- Optional accessories, including their simulation data. The rendering of these
+       into the final description is controlled by optenv variables, which default
+       each one to off.-->
+  <xacro:include filename="accessories.urdf.xacro" />
 </robot>

Commit message: Add xacro wrapper script to provide some pre-cooked "configs", especially for simulated Jackal.

File: urdf/accessories.urdf.xacro (robot description, xacro)
@@ -11,5 +11,6 @@
   <xacro:include filename="accessories/sick_lms1xx.urdf.xacro" />
   <xacro:if value="$(optenv JACKAL_LASER 0)">
-    <sick_lms1xx_mount prefix="$(optenv JACKAL_LASER_MOUNT front)" />
+    <sick_lms1xx_mount prefix="$(optenv JACKAL_LASER_MOUNT front)"
+                       topic="$(optenv JACKAL_LASER_TOPIC scan)" />
     <joint name="$front_laser_mount_joint" type="fixed">
       <origin xyz="$(optenv JACKAL_LASER_OFFSET 0 0 0)"

File: urdf/accessories/sick_lms1xx.urdf.xacro (robot description, xacro)
@@ -39,5 +39,5 @@
     </inertial>
   </xacro:macro>
-  <xacro:macro name="sick_lms1xx_mount" params="prefix">
+  <xacro:macro name="sick_lms1xx_mount" params="prefix topic">
     <link name="${prefix}_laser_mount">
       <visual>
@@ -101,5 +101,5 @@
         </ray>
         <plugin name="gazebo_ros_laser" filename="libgazebo_ros_laser.so">
-          <topicName>scan</topicName>
+          <topicName>${topic}</topicName>
           <frameName>${prefix}_laser</frameName>
         </plugin>

Commit message: Modified the accessories.urdf.xacro to include both the GPS and mount plate, including standoffs.

File: urdf/accessories.urdf.xacro (robot description, xacro)
@@ -9,4 +9,34 @@
     jackal_base/launch/base.launch
   -->
+  <xacro:macro name="standoff" params="name length parent *origin">
+    <link name="${name}">
+      <visual>
+        <origin xyz="0 0 ${length/2}" rpy="0 0 0" />
+        <geometry>
+          <cylinder radius="0.004" length="${length}" />
+        </geometry>
+        <material name="light_grey" />
+      </visual>
+    </link>
+    <joint name="${name}_joint" type="fixed">
+      <xacro:insert_block name="origin" />
+      <parent link="${parent}" />
+      <child link="${name}" />
+    </joint>
+  </xacro:macro>
+  <xacro:macro name="standoff_box" params="mount height">
+    <standoff name="${mount}_standoff0" length="${height}" parent="${mount}_mount">
+      <origin xyz="0.060 0.060 0" rpy="0 0 0"/>
+    </standoff>
+    <standoff name="${mount}_standoff1" length="${height}" parent="${mount}_mount">
+      <origin xyz="0.060 -0.060 0" rpy="0 0 0"/>
+    </standoff>
+    <standoff name="${mount}_standoff2" length="${height}" parent="${mount}_mount">
+      <origin xyz="-0.060 0.060 0" rpy="0 0 0"/>
+    </standoff>
+    <standoff name="${mount}_standoff3" length="${height}" parent="${mount}_mount">
+      <origin xyz="-0.060 -0.060 0" rpy="0 0 0"/>
+    </standoff>
+  </xacro:macro>
   <xacro:include filename="accessories/sick_lms1xx.urdf.xacro" />
   <xacro:if value="$(optenv JACKAL_LASER 0)">
@@ -18,4 +48,16 @@
       <parent link="$(optenv JACKAL_LASER_MOUNT front)_mount" />
       <child link="$(optenv JACKAL_LASER_MOUNT front)_laser_mount" />
+    </joint>
+  </xacro:if>
+  <xacro:include filename="accessories/novatel_smart6.urdf.xacro" />
+  <xacro:include filename="accessories/bridge_plate.urdf.xacro" />
+  <xacro:if value="$(optenv JACKAL_NAVSAT 0)">
+    <bridge_plate mount="$(optenv JACKAL_NAVSAT_MOUNT rear)"
+                  height="$(optenv JACKAL_NAVSAT_HEIGHT 0.12)" />
+    <novatel_smart6 prefix="$(optenv JACKAL_NAVSAT_MOUNT rear)"/>
+    <joint name="$(optenv JACKAL_NAVSAT_MOUNT rear)_navsat_joint" type="fixed">
+      <origin xyz="0 0 0" rpy="0 0 0" />
+      <parent link="$(optenv JACKAL_NAVSAT_MOUNT rear)_bridge" />
+      <child link="$(optenv JACKAL_NAVSAT_MOUNT rear)_navsat" />
     </joint>
   </xacro:if>

Commit message: Refactor standoffs to separate file, add comments.

File: urdf/accessories.urdf.xacro (robot description, xacro)
@@ -2,5 +2,5 @@
 <robot xmlns:xacro="http://www.ros.org/wiki/xacro">
   <!--
-    As you add to this xacro, please be aware that both the robot and
+    As you add to this URDF, please be aware that both the robot and
     simulation include it. You must retain compatibility with all of
     the following launch files:
@@ -9,34 +9,9 @@
     jackal_base/launch/base.launch
   -->
-  <xacro:macro name="standoff" params="name length parent *origin">
-    <link name="${name}">
-      <visual>
-        <origin xyz="0 0 ${length/2}" rpy="0 0 0" />
-        <geometry>
-          <cylinder radius="0.004" length="${length}" />
-        </geometry>
-        <material name="light_grey" />
-      </visual>
-    </link>
-    <joint name="${name}_joint" type="fixed">
-      <xacro:insert_block name="origin" />
-      <parent link="${parent}" />
-      <child link="${name}" />
-    </joint>
-  </xacro:macro>
-  <xacro:macro name="standoff_box" params="mount height">
-    <standoff name="${mount}_standoff0" length="${height}" parent="${mount}_mount">
-      <origin xyz="0.060 0.060 0" rpy="0 0 0"/>
-    </standoff>
-    <standoff name="${mount}_standoff1" length="${height}" parent="${mount}_mount">
-      <origin xyz="0.060 -0.060 0" rpy="0 0 0"/>
-    </standoff>
-    <standoff name="${mount}_standoff2" length="${height}" parent="${mount}_mount">
-      <origin xyz="-0.060 0.060 0" rpy="0 0 0"/>
-    </standoff>
-    <standoff name="${mount}_standoff3" length="${height}" parent="${mount}_mount">
-      <origin xyz="-0.060 -0.060 0" rpy="0 0 0"/>
-    </standoff>
-  </xacro:macro>
+  <!-- Macros to generate standoffs for offset payload mounting. -->
+  <xacro:include filename="accessories/standoffs.urdf.xacro" />
+  <!-- This optional plate mounts both the upgraded GPS and the Velodyne 3D LIDAR. -->
+  <xacro:include filename="accessories/bridge_plate.urdf.xacro" />
+  <!-- If enabled, generate the LASER payload (by default, a SICK LMS111). -->
   <xacro:include filename="accessories/sick_lms1xx.urdf.xacro" />
   <xacro:if value="$(optenv JACKAL_LASER 0)">
@@ -50,9 +25,9 @@
     </joint>
   </xacro:if>
+  <!-- If enabled, generate the upgraded Navsat payload (a Novatel Smart6). -->
   <xacro:include filename="accessories/novatel_smart6.urdf.xacro" />
-  <xacro:include filename="accessories/bridge_plate.urdf.xacro" />
   <xacro:if value="$(optenv JACKAL_NAVSAT 0)">
     <bridge_plate mount="$(optenv JACKAL_NAVSAT_MOUNT rear)"
-                  height="$(optenv JACKAL_NAVSAT_HEIGHT 0.12)" />
+                  height="$(optenv JACKAL_NAVSAT_HEIGHT 0.1)" />
     <novatel_smart6 prefix="$(optenv JACKAL_NAVSAT_MOUNT rear)"/>
     <joint name="$(optenv JACKAL_NAVSAT_MOUNT rear)_navsat_joint" type="fixed">

File: urdf/accessories/novatel_smart6.urdf.xacro (robot description, xacro)
@@ -8,6 +8,6 @@
         <mesh filename="package://jackal_description/meshes/novatel-smart6.stl"/>
       </geometry>
-      <material name="white">
-        <color rgba="255 255 255 .9"/>
+      <material name="novatel_white">
+        <color rgba="0.8 0.8 0.8 1.0" />
       </material>
     </visual>

Commit message: Added Sick LMS1XX URDF.

File: urdf/accessories.urdf.xacro (robot description, xacro)
@@ -14,8 +14,8 @@
   <xacro:include filename="accessories/bridge_plate.urdf.xacro" />
   <!-- If enabled, generate the LASER payload (by default, a SICK LMS111). -->
-  <xacro:include filename="accessories/sick_lms1xx.urdf.xacro" />
+  <xacro:include filename="accessories/sick_lms1xx_mount.urdf.xacro" />
   <xacro:if value="$(optenv JACKAL_LASER 0)">
     <sick_lms1xx_mount prefix="$(optenv JACKAL_LASER_MOUNT front)"
-                       topic="$(optenv JACKAL_LASER_TOPIC scan)" />
+                       topic="$(optenv JACKAL_LASER_TOPIC front/scan)"/>
     <joint name="$front_laser_mount_joint" type="fixed">
       <origin xyz="$(optenv JACKAL_LASER_OFFSET 0 0 0)"

File: urdf/accessories/sick_lms1xx_mount.urdf.xacro (robot description, xacro)
@@ -26,18 +26,7 @@
 -->
 <robot xmlns:xacro="http://ros.org/wiki/xacro">
-  <xacro:property name="laser_x" value="0.105" />
-  <xacro:property name="laser_y" value="0.102" />
-  <xacro:property name="laser_z" value="0.152" />
-  <xacro:property name="laser_mass" value="1.1" />
-  <xacro:macro name="box_inertial" params="x y z mass">
-    <inertial>
-      <mass value="${mass}" />
-      <origin xyz="0 0 0" />
-      <inertia ixx="${0.0833333 * mass * (y*y + z*z)}" ixy="0.0" ixz="0.0"
-        iyy="${0.0833333 * mass * (x*x + z*z)}" iyz="0.0"
-        izz="${0.0833333 * mass * (x*x + y*y)}" />
-    </inertial>
-  </xacro:macro>
+  <xacro:include filename="$(find lms1xx)/urdf/sick_lms1xx.urdf.xacro" />
   <xacro:macro name="sick_lms1xx_mount" params="prefix topic">
+    <sick_lms1xx frame="${prefix}_laser" topic="${topic}" />
     <link name="${prefix}_laser_mount">
       <visual>
@@ -50,21 +39,4 @@
       </visual>
     </link>
-    <link name="${prefix}_laser">
-      <xacro:box_inertial x="${laser_x}" y="${laser_y}" z="${laser_z}" mass="${laser_mass}" />
-      <visual>
-        <origin xyz="0 0 0" rpy="0 0 0" />
-        <geometry>
-          <!-- Origin of this mesh is the focal point of the LIDAR. -->
-          <mesh filename="package://jackal_description/meshes/sick-lms1xx.stl" />
-        </geometry>
-        <material name="light_grey" />
-      </visual>
-      <collision>
-        <origin xyz="0 0 -0.05" rpy="0 0 0" />
-        <geometry>
-          <box size="${laser_x} ${laser_y} ${laser_z}" />
-        </geometry>
-      </collision>
-    </link>
     <joint name="${prefix}_laser_joint" type="fixed">
       <!-- This offset is from the base of the bracket to the LIDAR's focal point. -->
@@ -73,37 +45,4 @@
       <child link="${prefix}_laser" />
     </joint>
-    <gazebo reference="${prefix}_laser">
-      <material>Gazebo/Grey</material>
-      <turnGravityOff>true</turnGravityOff>
-      <sensor type="ray" name="${prefix}_laser">
-        <pose>0 0 0 0 0 0</pose>
-        <visualize>false</visualize>
-        <update_rate>40</update_rate>
-        <ray>
-          <scan>
-            <horizontal>
-              <samples>720</samples>
-              <resolution>1</resolution>
-              <min_angle>-1.570796</min_angle>
-              <max_angle>1.570796</max_angle>
-            </horizontal>
-          </scan>
-          <range>
-            <min>0.10</min>
-            <max>30.0</max>
-            <resolution>0.01</resolution>
-          </range>
-          <noise>
-            <type>gaussian</type>
-            <mean>0.0</mean>
-            <stddev>0.001</stddev>
-          </noise>
-        </ray>
-        <plugin name="gazebo_ros_laser" filename="libgazebo_ros_laser.so">
-          <topicName>${topic}</topicName>
-          <frameName>${prefix}_laser</frameName>
-        </plugin>
-      </sensor>
-    </gazebo>
   </xacro:macro>
 </robot>

Commit message: Fixed laser joint name.

File: urdf/accessories.urdf.xacro (robot description, xacro)
@@ -18,5 +18,5 @@
     <sick_lms1xx_mount prefix="$(optenv JACKAL_LASER_MOUNT front)"
                        topic="$(optenv JACKAL_LASER_TOPIC front/scan)"/>
-    <joint name="$front_laser_mount_joint" type="fixed">
+    <joint name="$(optenv JACKAL_LASER_MOUNT front)_laser_mount_joint" type="fixed">
       <origin xyz="$(optenv JACKAL_LASER_OFFSET 0 0 0)"
               rpy="$(optenv JACKAL_LASER_RPY 0 0 0)" />

Commit message: Added pointgrey camera accessories.

File: urdf/accessories.urdf.xacro (robot description, xacro)
@@ -18,5 +18,5 @@
     <sick_lms1xx_mount prefix="$(optenv JACKAL_LASER_MOUNT front)"
                        topic="$(optenv JACKAL_LASER_TOPIC front/scan)"/>
-    <joint name="$front_laser_mount_joint" type="fixed">
+    <joint name="$(optenv JACKAL_LASER_MOUNT front)_laser_mount_joint" type="fixed">
       <origin xyz="$(optenv JACKAL_LASER_OFFSET 0 0 0)"
               rpy="$(optenv JACKAL_LASER_RPY 0 0 0)" />
@@ -37,26 +37,27 @@
     </joint>
   </xacro:if>
-  <!--
-  <xacro:include filename="accessories/point_grey_flea.urdf.xacro" />
-  <xacro:if value="$(arg camera)">
-    <xacro:point_grey_flea3
-      prefix="front"
-      joint_parent="front_mount"
-      joint_xyz="0.135 0 0.015"
-      joint_rpy="0 0 0"
-      camera_x="0.0754"
-      camera_y="0.029"
-      camera_z="0.035"
-      camera_mass="0.085"
-      hfov="1.0471975512"
-      width="640"
-      height="512"
-      format="R8G8B8"
-      near="0.1"
-      far="300"
-      ns="jackal"
-      frame_id="front_mount"
-      />
+  <!-- If enabled, generate the flea3 camera payload. -->
+  <xacro:include filename="accessories/pointgrey_flea3_mount.urdf.xacro" />
+  <xacro:if value="$(optenv JACKAL_FLEA3 0)">
+    <pointgrey_flea3_mount prefix="$(optenv JACKAL_FLEA_MOUNT front)"
+                       name="$(optenv JACKAL_FLEA_NAME front)"/>
+    <joint name="$(optenv JACKAL_FLEA3_MOUNT front)_camera_mount_joint" type="fixed">
+      <origin xyz="$(optenv JACKAL_FLEA3_OFFSET 0 0 0)"
+              rpy="$(optenv JACKAL_FLEA3_RPY 0 0 0)" />
+      <parent link="$(optenv JACKAL_FLEA_MOUNT front)_mount" />
+      <child link="$(optenv JACKAL_FLEA_MOUNT front)_camera_mount" />
+    </joint>
   </xacro:if>
-  -->
+  <!-- If enabled, generate the bumblebee2 camera payload. -->
+  <xacro:include filename="accessories/pointgrey_bumblebee2_mount.urdf.xacro" />
+  <xacro:if value="$(optenv JACKAL_BB2 0)">
+    <pointgrey_bumblebee2_mount prefix="$(optenv JACKAL_BB2_MOUNT front)"
+                       name="$(optenv JACKAL_BB2_NAME front)"/>
+    <joint name="$(optenv JACKAL_BB2_MOUNT front)_camera_mount_joint" type="fixed">
+      <origin xyz="$(optenv JACKAL_BB2_OFFSET 0 0 0)"
+              rpy="$(optenv JACKAL_BB2_RPY 0 0 0)" />
+      <parent link="$(optenv JACKAL_BB2_MOUNT front)_mount" />
+      <child link="$(optenv JACKAL_BB2_MOUNT front)_camera_mount" />
+    </joint>
+  </xacro:if>
 </robot>
