Commit message: Added tilting option to point grey mount.

File: urdf/accessories.urdf.xacro (robot description, xacro)
@@ -37,9 +37,10 @@
     </joint>
   </xacro:if>
-  <!-- If enabled, generate the flea3 camera payload. -->
+  <!-- If enabled, generate the flea3 camera payload with a tilt of 30 degrees. -->
   <xacro:include filename="accessories/pointgrey_flea3_mount.urdf.xacro" />
   <xacro:if value="$(optenv JACKAL_FLEA3 0)">
     <pointgrey_flea3_mount prefix="$(optenv JACKAL_FLEA_MOUNT front)"
-                       name="$(optenv JACKAL_FLEA_NAME front)"/>
+                       name="$(optenv JACKAL_FLEA_NAME front)"
+                       tilt="$(optenv JACKAL_FLEA_TILT 0.5236)"/>
     <joint name="$(optenv JACKAL_FLEA3_MOUNT front)_camera_mount_joint" type="fixed">
       <origin xyz="$(optenv JACKAL_FLEA3_OFFSET 0 0 0)"
@@ -49,9 +50,10 @@
     </joint>
   </xacro:if>
-  <!-- If enabled, generate the bumblebee2 camera payload. -->
+  <!-- If enabled, generate the bumblebee2 camera payload with a tilt of 0 degrees. -->
   <xacro:include filename="accessories/pointgrey_bumblebee2_mount.urdf.xacro" />
   <xacro:if value="$(optenv JACKAL_BB2 0)">
     <pointgrey_bumblebee2_mount prefix="$(optenv JACKAL_BB2_MOUNT front)"
-                       name="$(optenv JACKAL_BB2_NAME front)"/>
+                       name="$(optenv JACKAL_BB2_NAME front)"
+                        tilt="$(optenv JACKAL_BB2_TILT 0)"/>
     <joint name="$(optenv JACKAL_BB2_MOUNT front)_camera_mount_joint" type="fixed">
       <origin xyz="$(optenv JACKAL_BB2_OFFSET 0 0 0)"

File: urdf/accessories/pointgrey_bumblebee2_mount.urdf.xacro (robot description, xacro)
@@ -1,9 +1,9 @@
 <robot xmlns:xacro="http://ros.org/wiki/xacro">
   <xacro:include filename="$(find pointgrey_camera_description)/urdf/pointgrey_bumblebee2.urdf.xacro" />
-  <xacro:macro name="pointgrey_bumblebee2_mount" params="prefix name">
+  <xacro:macro name="pointgrey_bumblebee2_mount" params="prefix name tilt">
     <BB2-08S2C-38 frame="${prefix}_camera" name="${name}" />
     <link name="${prefix}_camera_mount">
       <visual>
-        <origin xyz="0 0 0" rpy="1.57 0 1.57" />
+        <origin xyz="0 0 0" rpy="1.5707 0 1.5707" />
         <geometry>
           <!-- Origin of this mesh is the base of the mount. -->
@@ -13,9 +13,30 @@
       </visual>
     </link>
-    <joint name="${prefix}_camera_joint" type="fixed">
-      <origin xyz="0.1013 0 0.0318" rpy="0 0 0" />
+    <link name="${prefix}_camera_beam">
+      <visual>
+        <origin xyz="0 -.080 0.004" rpy="1.5707 0 1.5707" />
+        <geometry>
+          <!-- Origin of this mesh is the base of the mount. -->
+          <mesh filename="package://jackal_description/meshes/pointgrey-camera-beam.stl" scale="0.001 0.001 0.001" />
+        </geometry>
+        <material name="dark_grey" />
+      </visual>
+    </link>
+    <joint name="${prefix}_camera_pivot_joint" type="fixed">
+      <origin xyz="0.095 0 -0.002" rpy="0 ${tilt} 0" />
       <parent link="${prefix}_camera_mount" />
+      <child link="${prefix}_camera_beam" />
+    </joint>
+    <joint name="${prefix}_camera_bracket_joint" type="fixed">
+      <origin xyz="0.007 0 0.03450" rpy="0 0 0" />
+      <parent link="${prefix}_camera_beam" />
       <child link="${prefix}_camera" />
     </joint>
+    <gazebo reference="${prefix}_camera_beam">
+      <material>Gazebo/DarkGrey</material>
+    </gazebo>
+    <gazebo reference="${prefix}_camera_mount">
+      <material>Gazebo/DarkGrey</material>
+    </gazebo>
   </xacro:macro>
 </robot>

File: urdf/accessories/pointgrey_flea3_mount.urdf.xacro (robot description, xacro)
@@ -1,9 +1,9 @@
 <robot xmlns:xacro="http://ros.org/wiki/xacro">
   <xacro:include filename="$(find pointgrey_camera_description)/urdf/pointgrey_flea3.urdf.xacro" />
-  <xacro:macro name="pointgrey_flea3_mount" params="prefix name">
+  <xacro:macro name="pointgrey_flea3_mount" params="prefix name tilt:=0">
     <pointgrey_flea3 frame="${prefix}_camera" name="${name}" camera_x="0.0754" camera_y="0.029" camera_z="0.035" camera_mass="0.085" hfov="1.0471975512" fps="60" width="640" height="512"/>
     <link name="${prefix}_camera_mount">
       <visual>
-        <origin xyz="0 0 0" rpy="1.57 0 1.57" />
+        <origin xyz="0 0 0" rpy="1.5707 0 1.5707" />
         <geometry>
           <!-- Origin of this mesh is the base of the mount. -->
@@ -13,9 +13,30 @@
       </visual>
     </link>
-    <joint name="${prefix}_camera_joint" type="fixed">
-      <origin xyz="0.125 0 0.03175" rpy="0 0 0" />
+    <link name="${prefix}_camera_beam">
+      <visual>
+        <origin xyz="0 0 0" rpy="0 0 1.5707" />
+        <geometry>
+          <!-- Origin of this mesh is the base of the mount. -->
+          <mesh filename="package://jackal_description/meshes/pointgrey-camera-beam.stl" scale="0.001 0.001 0.001" />
+        </geometry>
+        <material name="dark_grey" />
+      </visual>
+    </link>
+    <joint name="${prefix}_camera_pivot_joint" type="fixed">
+      <origin xyz="0.102 0 0.008" rpy="0 ${tilt} 0" />
       <parent link="${prefix}_camera_mount" />
+      <child link="${prefix}_camera_beam" />
+    </joint>
+    <joint name="${prefix}_camera_bracket_joint" type="fixed">
+      <origin xyz="0.020 0 0.0245" rpy="0 0 0" />
+      <parent link="${prefix}_camera_beam" />
       <child link="${prefix}_camera" />
     </joint>
+    <gazebo reference="${prefix}_camera_beam">
+      <material>Gazebo/DarkGrey</material>
+    </gazebo>
+    <gazebo reference="${prefix}_camera_mount">
+      <material>Gazebo/DarkGrey</material>
+    </gazebo>
   </xacro:macro>
 </robot>

File: urdf/accessories/sick_lms1xx_mount.urdf.xacro (robot description, xacro)
@@ -45,4 +45,7 @@
       <child link="${prefix}_laser" />
     </joint>
+    <gazebo reference="${prefix}_laser_mount">
+      <material>Gazebo/DarkGrey</material>
+    </gazebo>
   </xacro:macro>
 </robot>

Commit message: Unified camera mount and added example for customization without using envvar scheme.

File: urdf/accessories.urdf.xacro (robot description, xacro)
@@ -38,8 +38,8 @@
   </xacro:if>
   <!-- If enabled, generate the flea3 camera payload with a tilt of 30 degrees. -->
-  <xacro:include filename="accessories/pointgrey_flea3_mount.urdf.xacro" />
+  <xacro:include filename="accessories/camera_mount.urdf.xacro" />
+  <xacro:include filename="$(find pointgrey_camera_description)/urdf/pointgrey_flea3.urdf.xacro" />
   <xacro:if value="$(optenv JACKAL_FLEA3 0)">
-    <pointgrey_flea3_mount prefix="$(optenv JACKAL_FLEA_MOUNT front)"
-                       name="$(optenv JACKAL_FLEA_NAME front)"
+    <camera_mount prefix="$(optenv JACKAL_FLEA_MOUNT front)"
                        tilt="$(optenv JACKAL_FLEA_TILT 0.5236)"/>
     <joint name="$(optenv JACKAL_FLEA3_MOUNT front)_camera_mount_joint" type="fixed">
@@ -49,10 +49,18 @@
       <child link="$(optenv JACKAL_FLEA_MOUNT front)_camera_mount" />
     </joint>
+    <pointgrey_flea3 frame="$(optenv JACKAL_FLEA3_MOUNT front)_camera" name="$(optenv JACKAL_FLEA_NAME front)"
+      camera_x="0.0754" camera_y="0.029" camera_z="0.035"
+      camera_mass="0.085" hfov="1.0471975512" fps="60" width="640" height="512"/>
+    <joint name="$(optenv JACKAL_FLEA3_MOUNT front)_camera_bracket_joint" type="fixed">
+      <origin xyz="0.020 0 0.0245" rpy="0 0 0" />
+      <parent link="$(optenv JACKAL_FLEA3_MOUNT front)_camera_beam" />
+      <child link="$(optenv JACKAL_FLEA3_MOUNT front)_camera" />
+    </joint>
   </xacro:if>
   <!-- If enabled, generate the bumblebee2 camera payload with a tilt of 0 degrees. -->
-  <xacro:include filename="accessories/pointgrey_bumblebee2_mount.urdf.xacro" />
+  <xacro:include filename="accessories/camera_mount.urdf.xacro" />
+  <xacro:include filename="$(find pointgrey_camera_description)/urdf/pointgrey_bumblebee2.urdf.xacro" />
   <xacro:if value="$(optenv JACKAL_BB2 0)">
-    <pointgrey_bumblebee2_mount prefix="$(optenv JACKAL_BB2_MOUNT front)"
-                       name="$(optenv JACKAL_BB2_NAME front)"
+    <camera_mount prefix="$(optenv JACKAL_BB2_MOUNT front)"
                         tilt="$(optenv JACKAL_BB2_TILT 0)"/>
     <joint name="$(optenv JACKAL_BB2_MOUNT front)_camera_mount_joint" type="fixed">
@@ -62,4 +70,10 @@
       <child link="$(optenv JACKAL_BB2_MOUNT front)_camera_mount" />
     </joint>
+    <BB2-08S2C-38 frame="$(optenv JACKAL_BB2_MOUNT front)_camera" name="$(optenv JACKAL_BB2_NAME front)" />
+    <joint name="$(optenv JACKAL_BB2_MOUNT front)_camera_bracket_joint" type="fixed">
+      <origin xyz="0.007 0 0.02450" rpy="0 0 0" />
+      <parent link="$(optenv JACKAL_BB2_MOUNT front)_camera_beam" />
+      <child link="$(optenv JACKAL_BB2_MOUNT front)_camera" />
+    </joint>
   </xacro:if>
 </robot>

Commit message: Added stereo camera accessory.

File: urdf/accessories.urdf.xacro (robot description, xacro)
@@ -37,7 +37,8 @@
     </joint>
   </xacro:if>
-  <!-- If enabled, generate the flea3 camera payload with a tilt of 30 degrees. -->
+  <!-- Common camera mounts and accessory URDFs. -->
   <xacro:include filename="$(find jackal_description)/urdf/accessories/camera_mount.urdf.xacro" />
   <xacro:include filename="$(find pointgrey_camera_description)/urdf/pointgrey_flea3.urdf.xacro" />
+  <!-- If enabled, generate the flea3 camera payload with a tilt of 30 degrees. -->
   <xacro:if value="$(optenv JACKAL_FLEA3 0)">
     <camera_mount prefix="$(optenv JACKAL_FLEA3_MOUNT front)"
@@ -50,5 +51,5 @@
     </joint>
     <pointgrey_flea3 frame="$(optenv JACKAL_FLEA3_MOUNT front)_camera" name="$(optenv JACKAL_FLEA3_NAME front)"
-      camera_x="0.0754" camera_y="0.029" camera_z="0.035"
+      camera_x="0.0754" camera_y="0.029" camera_z="0.029"
       camera_mass="0.085" hfov="1.0471975512" fps="60" width="640" height="512"/>
     <joint name="$(optenv JACKAL_FLEA3_MOUNT front)_camera_bracket_joint" type="fixed">
@@ -58,7 +59,35 @@
     </joint>
   </xacro:if>
+  <xacro:include filename="$(find jackal_description)/urdf/accessories/stereo_camera_mount.urdf.xacro" />
+  <!-- If enabled, generates a pair of flea3 cameras for stereo vision with a tilt of 30 degrees. -->
+  <xacro:if value="$(optenv JACKAL_STEREO_FLEA3 0)">
+    <stereo_camera_mount prefix="$(optenv JACKAL_FLEA3_MOUNT front)"
+                       tilt="$(optenv JACKAL_FLEA3_TILT 0.5236)"/>
+    <joint name="$(optenv JACKAL_FLEA3_MOUNT front)_stereo_camera_mount_joint" type="fixed">
+      <origin xyz="$(optenv JACKAL_FLEA3_OFFSET 0 0 0)"
+              rpy="$(optenv JACKAL_FLEA3_RPY 0 0 0)" />
+      <parent link="$(optenv JACKAL_FLEA3_MOUNT front)_mount" />
+      <child link="$(optenv JACKAL_FLEA3_MOUNT front)_stereo_camera_mount" />
+    </joint>
+    <pointgrey_flea3 frame="$(optenv JACKAL_FLEA3_MOUNT front)_left_camera" name="$(optenv JACKAL_FLEA3_LEFT_NAME front/left)"
+      camera_x="0.0754" camera_y="0.029" camera_z="0.029"
+      camera_mass="0.085" hfov="1.0471975512" fps="60" width="640" height="512"/>
+    <joint name="$(optenv JACKAL_FLEA3_MOUNT front)_left_stereo_camera_bracket_joint" type="fixed">
+      <origin xyz="0.015 $(optenv JACKAL_STEREO_SEPERATION 0.16) 0.0599" rpy="0 0 0" />
+      <parent link="$(optenv JACKAL_FLEA3_MOUNT front)_stereo_camera_beam" />
+      <child link="$(optenv JACKAL_FLEA3_MOUNT front)_left_camera" />
+    </joint>
+    <pointgrey_flea3 frame="$(optenv JACKAL_FLEA3_MOUNT front)_right_camera" name="$(optenv JACKAL_FLEA3_RIGHT_NAME front/right)"
+      camera_x="0.0754" camera_y="0.029" camera_z="0.029"
+      camera_mass="0.085" hfov="1.0471975512" fps="60" width="640" height="512"/>
+    <joint name="$(optenv JACKAL_FLEA3_MOUNT front)_right_stereo_camera_bracket_joint" type="fixed">
+      <origin xyz="0.015 -$(optenv JACKAL_STEREO_SEPERATION 0.16) 0.0599" rpy="0 0 0" />
+      <parent link="$(optenv JACKAL_FLEA3_MOUNT front)_stereo_camera_beam" />
+      <child link="$(optenv JACKAL_FLEA3_MOUNT front)_right_camera" />
+    </joint>
+  </xacro:if>
   <!-- If enabled, generate the bumblebee2 camera payload with a tilt of 0 degrees. -->
-  <xacro:include filename="$(find jackal_description)/urdf/accessories/camera_mount.urdf.xacro" />
   <xacro:include filename="$(find pointgrey_camera_description)/urdf/pointgrey_bumblebee2.urdf.xacro" />
+  <!-- If enabled, generate the bumblebee2 camera payload with a tilt of 0 degrees. -->
   <xacro:if value="$(optenv JACKAL_BB2 0)">
     <camera_mount prefix="$(optenv JACKAL_BB2_MOUNT front)"

Commit message: Make urdf refer explicitly to jackal_description, rather than relying on current working directory being correct, for easier external includes

File: urdf/accessories.urdf.xacro (robot description, xacro)
@@ -10,9 +10,9 @@
   -->
   <!-- Macros to generate standoffs for offset payload mounting. -->
-  <xacro:include filename="accessories/standoffs.urdf.xacro" />
+  <xacro:include filename="$(find jackal_description)/urdf/accessories/standoffs.urdf.xacro" />
   <!-- This optional plate mounts both the upgraded GPS and the Velodyne 3D LIDAR. -->
-  <xacro:include filename="accessories/bridge_plate.urdf.xacro" />
+  <xacro:include filename="$(find jackal_description)/urdf/accessories/bridge_plate.urdf.xacro" />
   <!-- If enabled, generate the LASER payload (by default, a SICK LMS111). -->
-  <xacro:include filename="accessories/sick_lms1xx_mount.urdf.xacro" />
+  <xacro:include filename="$(find jackal_description)/urdf/accessories/sick_lms1xx_mount.urdf.xacro" />
   <xacro:if value="$(optenv JACKAL_LASER 0)">
     <sick_lms1xx_mount prefix="$(optenv JACKAL_LASER_MOUNT front)"
@@ -26,5 +26,5 @@
   </xacro:if>
   <!-- If enabled, generate the upgraded Navsat payload (a Novatel Smart6). -->
-  <xacro:include filename="accessories/novatel_smart6.urdf.xacro" />
+  <xacro:include filename="$(find jackal_description)/urdf/accessories/novatel_smart6.urdf.xacro" />
   <xacro:if value="$(optenv JACKAL_NAVSAT 0)">
     <bridge_plate mount="$(optenv JACKAL_NAVSAT_MOUNT rear)"
@@ -38,5 +38,5 @@
   </xacro:if>
   <!-- If enabled, generate the flea3 camera payload with a tilt of 30 degrees. -->
-  <xacro:include filename="accessories/camera_mount.urdf.xacro" />
+  <xacro:include filename="$(find jackal_description)/urdf/accessories/camera_mount.urdf.xacro" />
   <xacro:include filename="$(find pointgrey_camera_description)/urdf/pointgrey_flea3.urdf.xacro" />
   <xacro:if value="$(optenv JACKAL_FLEA3 0)">
@@ -59,5 +59,5 @@
   </xacro:if>
   <!-- If enabled, generate the bumblebee2 camera payload with a tilt of 0 degrees. -->
-  <xacro:include filename="accessories/camera_mount.urdf.xacro" />
+  <xacro:include filename="$(find jackal_description)/urdf/accessories/camera_mount.urdf.xacro" />
   <xacro:include filename="$(find pointgrey_camera_description)/urdf/pointgrey_bumblebee2.urdf.xacro" />
   <xacro:if value="$(optenv JACKAL_BB2 0)">

File: urdf/jackal.urdf.xacro (robot description, xacro)
@@ -13,4 +13,5 @@
   <xacro:property name="dummy_inertia" value="1e-09"/>
   <xacro:property name="mount_spacing" value="0.120" />
+  <xacro:property name="jackal_description_dir" value="$(find jackal_description)" />
   <material name="dark_grey"><color rgba="0.2 0.2 0.2 1.0" /></material>
   <material name="light_grey"><color rgba="0.4 0.4 0.4 1.0" /></material>
@@ -167,10 +168,12 @@
   </joint>
   <!-- Bring in simulation data for Gazebo. -->
-  <xacro:include filename="jackal.gazebo" />
+  <xacro:include filename="$(find jackal_description)/urdf/jackal.gazebo" />
   <!-- Optional standard accessories, including their simulation data. The rendering
        of these into the final description is controlled by optenv variables, which
        default each one to off.-->
-  <xacro:include filename="accessories.urdf.xacro" />
+  <xacro:include filename="$(find jackal_description)/urdf/accessories.urdf.xacro" />
   <!-- Optional custom includes. -->
-  <xacro:include filename="$(optenv JACKAL_URDF_EXTRAS empty.urdf)" />
+  <xacro:if value="$(optenv JACKAL_URDF_EXTRAS 0)">
+    <xacro:include filename="$(env JACKAL_URDF_EXTRAS)" />
+  </xacro:if>
 </robot>

Commit message: Modify the hokuyo accessory so that it works properly in gazebo/rviz.  Add an additional environment var JACKAL_LASER_HOKUYO which overrides the default lms1xx sensor with the ust10.

File: urdf/accessories.urdf.xacro (robot description, xacro)
@@ -15,13 +15,26 @@
   <!-- If enabled, generate the LASER payload (by default, a SICK LMS111). -->
   <xacro:if value="$(optenv JACKAL_LASER 0)">
-    <xacro:include filename="$(find jackal_description)/urdf/accessories/sick_lms1xx_mount.urdf.xacro" />
-    <sick_lms1xx_mount prefix="$(optenv JACKAL_LASER_MOUNT front)"
-                       topic="$(optenv JACKAL_LASER_TOPIC front/scan)"/>
-    <joint name="$(optenv JACKAL_LASER_MOUNT front)_laser_mount_joint" type="fixed">
-      <origin xyz="$(optenv JACKAL_LASER_OFFSET 0 0 0)"
-              rpy="$(optenv JACKAL_LASER_RPY 0 0 0)" />
-      <parent link="$(optenv JACKAL_LASER_MOUNT front)_mount" />
-      <child link="$(optenv JACKAL_LASER_MOUNT front)_laser_mount" />
-    </joint>
+    <xacro:if value="$(optenv JACKAL_LASER_HOKUYO 0)">
+      <xacro:include filename="$(find jackal_description)/urdf/accessories/hokuyo_ust10.urdf.xacro" />
+      <hokuyo_ust10_mount prefix="$(optenv JACKAL_LASER_MOUNT front)"
+                          topic="$(optenv JACKAL_LASER_TOPIC front/scan)" />
+      <joint name="$(optenv JACKAL_LASER_MOUNT front)_laser_mount_joint" type="fixed">
+        <origin xyz="$(optenv JACKAL_LASER_OFFSET 0.11 0 0)"
+                rpy="$(optenv JACKAL_LASER_RPY 0 0 0)" />
+        <parent link="$(optenv JACKAL_LASER_MOUNT front)_mount" />
+        <child link="$(optenv JACKAL_LASER_MOUNT front)_laser_mount" />
+      </joint>
+    </xacro:if>
+    <xacro:unless value="$(optenv JACKAL_LASER_HOKUYO 0)">
+      <xacro:include filename="$(find jackal_description)/urdf/accessories/sick_lms1xx_mount.urdf.xacro" />
+      <sick_lms1xx_mount prefix="$(optenv JACKAL_LASER_MOUNT front)"
+                         topic="$(optenv JACKAL_LASER_TOPIC front/scan)"/>
+      <joint name="$(optenv JACKAL_LASER_MOUNT front)_laser_mount_joint" type="fixed">
+        <origin xyz="$(optenv JACKAL_LASER_OFFSET 0 0 0)"
+                rpy="$(optenv JACKAL_LASER_RPY 0 0 0)" />
+        <parent link="$(optenv JACKAL_LASER_MOUNT front)_mount" />
+        <child link="$(optenv JACKAL_LASER_MOUNT front)_laser_mount" />
+      </joint>
+    </xacro:unless>
   </xacro:if>
   <!-- If enabled, generate the upgraded Navsat payload (a Novatel Smart6). -->
